File: calc-v2.kicad_sch (KiCad schematic)
At the start: 79 parts, among them J1 USB_C_Receptacle_USB2.0_16P, SW1 SW_Push_45deg, SW10 SW_Push_45deg, SW11 SW_Push_45deg, SW12 SW_Push_45deg, SW13 SW_Push_45deg, SW14 SW_Push_45deg, SW15 SW_Push_45deg, SW16 SW_Push_45deg, SW17 SW_Push_45deg, SW18 SW_Push_45deg, SW19 SW_Push_45deg, SW2 SW_Push_45deg, SW20 SW_Push_45deg, SW21 SW_Push_45deg, SW22 SW_Push_45deg, SW23 SW_Push_45deg, SW24 SW_Push_45deg, SW25 SW_Push_45deg, SW26 SW_Push_45deg, SW27 SW_Push_45deg, SW28 SW_Push_45deg, SW29 SW_Push_45deg, SW3 SW_Push_45deg, SW30 SW_Push_45deg, SW31 SW_Push_45deg, SW32 SW_Push_45deg, SW33 SW_Push_45deg, SW34 SW_Push_45deg, SW35 SW_Push_45deg, SW36 SW_Push_45deg, SW37 SW_Push_45deg, SW38 SW_Push_45deg, SW39 SW_Push_45deg, SW4 SW_Push_45deg, SW40 SW_Push_45deg, SW41 SW_Push_45deg, SW42 SW_Push_45deg, SW43 SW_Push_45deg, SW44 SW_Push_45deg, SW45 SW_Push_45deg, SW46 SW_Push_45deg, SW47 SW_Push_45deg, SW48 SW_Push_45deg, SW5 SW_Push_45deg, SW6 SW_Push_45deg, SW7 SW_Push_45deg, SW8 SW_Push_45deg, SW9 SW_Push_45deg, U1 RP2350_60QFN, Y1 ABM8-272-T3

Commit message: more
Parts:
- removed H1, H2, H3, H4: MountingHole, symbol Mechanical:MountingHole
- added C18, C19, C20, C21: 4.7u, symbol Device:C
- added U2: NCP1117-1.5_SOT223, Package_TO_SOT_SMD:SOT-223-3_TabPin2, symbol Regulator_Linear:NCP1117-1.5_SOT223
- renumbered C17 to C1, C7 to C10, C8 to C11, C9 to C12, C10 to C13, C11 to C14, C12 to C15, C13 to C16, C14 to C17, C4 to C2, C16 to C3, C19 to C4, C20 to C5, C3 to C6, C15 to C7, C5 to C8, C6 to C9, R3 to R1, R7 to R2, R4 to R3, R5 to R4, R1 to R5, R2 to R6, SW7 to SW10, SW13 to SW11, SW14 to SW12, SW23 to SW13, SW24 to SW14, SW39 to SW15, SW40 to SW16, SW3 to SW17, SW8 to SW18, SW15 to SW19, SW6 to SW2, SW16 to SW20, SW25 to SW21, SW26 to SW22, SW41 to SW23, SW42 to SW24, SW4 to SW25, SW9 to SW26, SW17 to SW27, SW18 to SW28, SW27 to SW29, SW11 to SW3, SW28 to SW30, SW43 to SW31, SW44 to SW32, SW5 to SW33, SW10 to SW34, SW19 to SW35, SW20 to SW36, SW29 to SW37, SW30 to SW38, SW45 to SW39, SW12 to SW4, SW46 to SW40, SW31 to SW41, SW32 to SW42, SW33 to SW43, SW34 to SW44, SW35 to SW45, SW36 to SW46, SW21 to SW5, SW22 to SW6, SW37 to SW7, SW38 to SW8, SW2 to SW9
Connections:
- net +3V3: now also C20.2, C21.1, U2.2 (VO)
- net GND: now also C18.2, C19.2, C20.1, C21.2; no longer J1.S1 (SHIELD)
- net VBUS: now also C18.1, C19.1, U2.3 (VI)
Other:
- note added: "conversion to 3v3"
- moved on the sheet: J1, R5, R6

Commit message: changes
Parts:
- removed L1: 3.3u, symbol Device:L
- removed U1: RP2350_60QFN, Package_DFN_QFN:QFN-60-1EP_7x7mm_P0.4mm_EP3.4x3.4mm, symbol RP2350:RP2350_60QFN
- removed U2: NCP1117-1.5_SOT223, Package_TO_SOT_SMD:SOT-223-3_TabPin2, symbol Regulator_Linear:NCP1117-1.5_SOT223
- added C24, C25, C28, C29, C30, C33: 4.7u, Capacitor_SMD:C_0402_1005Metric, symbol Device:C
- added C26, C27: 100n, Capacitor_SMD:C_0402_1005Metric, symbol Device:C
- added C31: 10u, Capacitor_SMD:C_0402_1005Metric, symbol Device:C
- added C32: 220n, Capacitor_SMD:C_0402_1005Metric, symbol Device:C
- added D5: D_Schottky, symbol Device:D_Schottky
- added DS1: E28GA-T-CW250-N, symbol AAAAAAA:E28GA-T-CW250-N
- added J2: Conn_01x02_MountingPin, symbol Connector_Generic_MountingPin:Conn_01x02_MountingPin
- added L1: AOTA-B201610S3R3-101-T, AAAAA:AOTAB201610S3R3101T, symbol AAAAAAA:AOTA-B201610S3R3-101-T
- added L2: 10u, symbol Device:L
- added R10, R17, R7: 10k, symbol Device:R
- added R11, R12, R13: 46k4, symbol Device:R
- added R14: 10, symbol Device:R
- added R15: 1k, Resistor_SMD:R_0402_1005Metric, symbol Device:R
- added R8: 2k, symbol Device:R
- added R9: 3.09k, symbol Device:R
- added SW49: SW_Push_45deg, symbol Switch:SW_Push_45deg
- added U1: W25Q128JVS, Package_SO:SOIC-8_5.3x5.3mm_P1.27mm, symbol Memory_Flash:W25Q128JVS
- added U2: NCP1117-3.3_SOT223, Package_TO_SOT_SMD:SOT-223-3_TabPin2, symbol Regulator_Linear:NCP1117-3.3_SOT223
- added U3: BQ24074RGT, Package_DFN_QFN:VQFN-16-1EP_3x3mm_P0.5mm_EP1.6x1.6mm, symbol Battery_Management:BQ24074RGT
- added U4: TPS61165DBV, Package_TO_SOT_SMD:SOT-23-6, symbol Driver_LED:TPS61165DBV
- added U5: RP2350B, Package_DFN_QFN:QFN-80-1EP_10x10mm_P0.4mm_EP3.4x3.4mm, symbol MCU_RaspberryPi:RP2350B
- added U6: APS6404L-3SQRx-ZR, Package_SON:Winbond_USON-8-1EP_3x2mm_P0.5mm_EP0.2x1.6mm, symbol Memory_RAM:APS6404L-3SQRx-ZR
Connections:
- net +1V1: now also L1.1, U5.10 (DVDD), U5.32 (DVDD), U5.51 (DVDD), U5.65 (VREG_FB)
- net +3V3: now also C8.1, C26.2, C27.2, C28.1, C29.2, DS1.8 (VDDI), DS1.9 (VDD), R10.2, R12.2, R13.1, R17.2, U1.8 (VCC), U2.2 (VO), U5.15 (IOVDD), U5.24 (IOVDD), U5.29 (IOVDD), U5.41 (IOVDD), U5.5 (IOVDD), U5.50 (IOVDD), U5.59 (ADC_AVDD), U5.60 (IOVDD), U5.64 (VREG_VIN), U5.68 (USB_OTP_VDD), U5.69 (QSPI_IOVDD), U5.76 (IOVDD), U6.8 (VDD); no longer C2.1
- net GND: now also J1.S1 (SHIELD), C24.2, C25.2, C26.1, C27.1, C28.2, C29.1, C30.2, C31.2, C32.1, C33.2, DS1.1 (GND), DS1.2 (GND), J2.2 (Pin_2), J2.MP (MountPin), R11.1, R14.2, R7.2, R8.1, R9.1, SW49.2, U1.4 (GND), U2.1 (GND), U3.17 (VSS), U3.4 (~{CE}), U3.5 (EN2), U3.8 (VSS), U4.4 (GND), U5.62 (VREG_PGND), U5.81 (GND), U6.4 (VSS)
- net RUN: now also U5.35 (RUN)
- net SWCLK: now also U5.33 (SWCLK)
- net SWD: now also U5.34 (SWDIO)
- net SW_C1: now also U5.7 (GPIO9)
- net SW_C2: now also U5.8 (GPIO10)
- net SW_C3: now also U5.9 (GPIO11)
- net SW_C4: now also U5.11 (GPIO12)
- net SW_C5: now also U5.12 (GPIO13)
- net SW_C6: now also U5.13 (GPIO14)
- net SW_R1: now also U5.78 (GPIO1)
- net SW_R2: now also U5.79 (GPIO2)
- net SW_R3: now also U5.80 (GPIO3)
- net SW_R4: now also U5.1 (GPIO4)
- net SW_R5: now also U5.2 (GPIO5)
- net SW_R6: now also U5.3 (GPIO6)
- net SW_R7: now also U5.4 (GPIO7)
- net SW_R8: now also U5.6 (GPIO8)
- net USB_DN: now also U5.66 (USB_DM)
- net USB_DP: now also U5.67 (USB_DP)
- net VBUS: now also C33.1; no longer C18.1, C19.1
- net XIN: now also U5.30 (XIN)
- net XOUT: now also U5.31 (XOUT)
- net Resistors should be close to microcontroller: now reaches J1.A5 (CC1), R5.1
- net at R1.2: now also C2.1, U5.61 (VREG_AVDD); no longer C8.1
- new net: R11.2, U3.14 (TMR)
- new net: D5.2 (A), L2.2, U4.3 (SW)
- new net: L1.2, U5.63 (VREG_LX)
- new net: C32.2, U4.5 (COMP)
- new net: R9.2, U3.12 (ILIM)
- new net: R15.2, SW49.1
- new net: R7.1, U3.1 (TS)
- new net: R8.2, U3.16 (ISET)
- new net +BATT: C25.1, J2.1 (Pin_1), U3.2 (BAT), U3.3 (BAT)
- new net BRIGHT_CTRL: U4.2 (CTRL)
- new net CHG: R12.1, U3.9 (~{CHG})
- new net FLASH_IO0: U1.5 (DI/IO_{0}), U5.72 (QSPI_SD0), U6.5 (SI/SIO0)
- new net FLASH_IO1: U1.2 (DO/IO_{1}), U5.74 (QSPI_SD1), U6.2 (SO/SIO1)
- new net FLASH_IO2: U1.3 (~{WP}/IO_{2}), U5.73 (QSPI_SD2), U6.3 (SIO2)
- new net FLASH_IO3: U1.7 (~{HOLD}/~{RESET}/IO_{3}), U5.70 (QSPI_SD3), U6.7 (SIO3)
- new net FLASH_SCLK: U1.6 (CLK), U5.71 (QSPI_SCLK), U6.6 (SCLK)
- new net FLASH_SS: R10.1, R15.1, U1.1 (~{CS}), U5.75 (~{QSPI_SS})
- new net LEDA: C31.1, D5.1 (K), DS1.40 (LEDA)
- new net LEDK: DS1.39 (LEDK), R14.1, U4.6 (FB)
- new net PGOOD: R13.2, U3.7 (~{PGOOD})
- new net PSRAM_SS: R17.1, U5.77 (GPIO0), U6.1 (~{CE})
- new net VSYS: C18.1, C19.1, C24.1, C30.1, L2.1, U2.3 (VI), U3.10 (OUT), U3.11 (OUT), U3.6 (EN1), U4.1 (VIN)
- no-connect marks 1 -> 35
Other:
- note added: "BQ24074RGT li-on charge management controller"
- note added: "FLASH"
- note added: "JST connector"
- note added: "PSRAM"
- note added: "Pull up for cs"
- note added: "RP2350 + decoupling"
- note added: "TPS61165DBV LED driver"
- note added: "cap rated for 25V"
- note added: "cap rated for 50V"
- note added: "d rated for 40V reverse"
- note added: "figure out which config you want for this controller"
- note added: "todo: maybe put a diode to protect?"
- moved on the sheet: C1, C18, C19, C20, C21, C3, C4, C5, C7, J1, R1, R2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

Commit message: more changes
Parts:
- removed SW1, SW10, SW11, SW12, SW13, SW14, SW15, SW16, SW17, SW18, SW19, SW2, SW20, SW21, SW22, SW23, SW24, SW25, SW26, SW27, SW28, SW29, SW3, SW30, SW31, SW32, SW33, SW34, SW35, SW36, SW37, SW38, SW39, SW4, SW40, SW41, SW42, SW43, SW44, SW45, SW46, SW47, SW48, SW5, SW6, SW7, SW8, SW9: SW_Push_45deg, symbol Switch:SW_Push_45deg
- added C34: 1u, Capacitor_SMD:C_0402_1005Metric, symbol Device:C
- added SW1, SW10, SW11, SW12, SW13, SW14, SW15, SW16, SW17, SW18, SW19, SW2, SW20, SW21, SW22, SW23, SW24, SW25, SW26, SW27, SW28, SW29, SW3, SW30, SW31, SW32, SW33, SW34, SW35, SW36, SW37, SW38, SW39, SW4, SW40, SW41, SW42, SW43, SW44, SW45, SW46, SW47, SW48, SW5, SW6, SW7, SW8, SW9: TS04-66-43-BK-100-SMT, AAAAA:SW_TS04-66-43-BK-100-SMT, symbol AAAAAAA:TS04-66-43-BK-100-SMT
- SW49: footprint (none) -> AAAAA:SW_TS04-66-43-BK-100-SMT
Connections:
- net +3V3: now also C34.2
- net GND: now also C34.1
- net SW_C1: now also SW1.1
- net SW_C2: now also SW2.1
- net SW_C3: now also SW3.1
- net SW_C4: now also SW4.1
- net SW_C5: now also SW5.1
- net SW_C6: now also SW6.1
- net SW_R1: now also SW1.4
- net SW_R2: now also SW7.4
- net SW_R3: now also SW13.4
- net SW_R4: now also SW19.4
- net SW_R5: now also SW25.4
- net SW_R6: now also SW31.4
- net SW_R7: now also SW37.4
- net SW_R8: now also SW43.4
- net VBUS: now also U3.13 (IN)
- new net: SW27.3, SW33.1
- new net: SW33.2, SW34.4
- new net: SW33.3, SW39.1
- new net: SW32.2, SW33.4
- new net: SW35.3, SW41.1
- new net: SW41.2, SW42.4
- new net: SW41.3, SW47.1
- new net: SW40.2, SW41.4
- new net: SW42.3, SW48.1
- new net: SW47.2, SW48.4
- new net: SW12.1, SW6.3
- new net: SW12.3, SW18.1
- new net: SW11.2, SW12.4
- new net: SW14.1, SW8.3
- new net: SW14.2, SW15.4
- new net: SW14.3, SW20.1
- new net: SW13.2, SW14.4
- new net: SW21.3, SW27.1
- new net: SW27.2, SW28.4
- new net: SW26.2, SW27.4
- new net: SW24.3, SW30.1
- new net: SW30.3, SW36.1
- new net: SW29.2, SW30.4
- new net: SW34.3, SW40.1
- new net: SW40.3, SW46.1
- new net: SW39.2, SW40.4
- new net: SW38.3, SW44.1
- new net: SW44.2, SW45.4
- new net: SW43.2, SW44.4
- new net: SW1.2, SW2.4
- new net: SW1.3, SW7.1
- new net: SW7.2, SW8.4
- new net: SW13.1, SW7.3
- new net: SW17.3, SW23.1
- new net: SW23.2, SW24.4
- new net: SW23.3, SW29.1
- new net: SW22.2, SW23.4
- new net: SW37.3, SW43.1
- new net: SW19.3, SW25.1
- new net: SW25.2, SW26.4
- new net: SW25.3, SW31.1
- new net: SW18.3, SW24.1
- new net: SW17.2, SW18.4
- new net: SW36.3, SW42.1
- new net: SW35.2, SW36.4
- new net: SW20.2, SW21.4
- new net: SW20.3, SW26.1
- new net: SW19.2, SW20.4
- new net: SW39.3, SW45.1
- new net: SW38.2, SW39.4
- new net: SW29.3, SW35.1
- new net: SW28.2, SW29.4
- new net: SW5.2, SW6.4
- new net: SW15.3, SW21.1
- new net: SW21.2, SW22.4
- new net: SW13.3, SW19.1
- new net: SW26.3, SW32.1
- new net: SW2.2, SW3.4
- new net: SW2.3, SW8.1
- new net: SW45.2, SW46.4
- new net: SW28.3, SW34.1
- new net: SW34.2, SW35.4
- new net: SW11.1, SW5.3
- new net: SW11.3, SW17.1
- new net: SW10.2, SW11.4
- new net: SW4.2, SW5.4
- new net: SW10.1, SW4.3
- new net: SW3.2, SW4.4
- new net: SW32.3, SW38.1
- new net: SW31.2, SW32.4
- new net: SW31.3, SW37.1
- new net: SW37.2, SW38.4
- new net: SW8.2, SW9.4
- new net: SW46.2, SW47.4
- new net: SW16.3, SW22.1
- new net: SW22.3, SW28.1
- new net: SW15.1, SW9.3
- new net: SW15.2, SW16.4
- new net: SW16.2, SW17.4
- new net: SW3.3, SW9.1
- new net: SW10.4, SW9.2
- new net: SW10.3, SW16.1
- no-connect marks 35 -> 49
Other:
- moved on the sheet: C33, R11

Commit message: components
Parts:
- removed SW1, SW10, SW11, SW12, SW13, SW14, SW15, SW16, SW17, SW18, SW19, SW2, SW20, SW21, SW22, SW23, SW24, SW25, SW26, SW27, SW28, SW29, SW3, SW30, SW31, SW32, SW33, SW34, SW35, SW36, SW37, SW38, SW39, SW4, SW40, SW41, SW42, SW43, SW44, SW45, SW46, SW47, SW48, SW5, SW6, SW7, SW8, SW9: TS04-66-43-BK-100-SMT, AAAAA:SW_TS04-66-43-BK-100-SMT, symbol AAAAAAA:TS04-66-43-BK-100-SMT
- added SW1, SW10, SW11, SW12, SW13, SW14, SW15, SW16, SW17, SW18, SW19, SW2, SW20, SW21, SW22, SW23, SW24, SW25, SW26, SW27, SW28, SW29, SW3, SW30, SW31, SW32, SW33, SW34, SW35, SW36, SW37, SW38, SW39, SW4, SW40, SW41, SW42, SW43, SW44, SW45, SW46, SW47, SW48, SW5, SW6, SW7, SW8, SW9: SW_Push_45deg, AAAAA:SW_TS04-66-43-BK-100-SMT, symbol Switch:SW_Push_45deg
Connections:
- net GND: now also U6.9 (EPAD)
- net SW_C1: now also SW1.1, SW13.1, SW19.1, SW25.1, SW31.1, SW37.1, SW43.1, SW7.1
- net SW_C2: now also SW14.1, SW2.1, SW20.1, SW26.1, SW32.1, SW38.1, SW44.1, SW8.1
- net SW_C3: now also SW15.1, SW21.1, SW27.1, SW3.1, SW33.1, SW39.1, SW45.1, SW9.1
- net SW_C4: now also SW10.1, SW16.1, SW22.1, SW28.1, SW34.1, SW4.1, SW40.1, SW46.1
- net SW_C5: now also SW11.1, SW17.1, SW23.1, SW29.1, SW35.1, SW41.1, SW47.1, SW5.1
- net SW_R1: now also SW1.2, SW2.2, SW3.2, SW4.2, SW5.2, SW6.2
- net SW_R2: now also SW10.2, SW11.2, SW12.2, SW7.2, SW8.2, SW9.2
- net SW_R3: now also SW13.2, SW14.2, SW15.2, SW16.2, SW17.2, SW18.2
- net SW_R4: now also SW19.2, SW20.2, SW21.2, SW22.2, SW23.2, SW24.2
- net SW_R5: now also SW25.2, SW26.2, SW27.2, SW28.2, SW29.2, SW30.2
- net SW_R6: now also SW31.2, SW32.2, SW33.2, SW34.2, SW35.2, SW36.2
- net SW_R7: now also SW37.2, SW38.2, SW39.2, SW40.2, SW41.2, SW42.2
- net SW_R8: now also SW43.2, SW44.2, SW45.2, SW46.2, SW47.2, SW48.2
- new net: SW12.1, SW18.1, SW24.1, SW30.1, SW36.1, SW42.1, SW48.1, SW6.1
- no-connect marks 49 -> 35

Commit message: ers
Parts:
- removed C18, C19, C20, C21: 4.7u, symbol Device:C
- removed U2: NCP1117-3.3_SOT223, Package_TO_SOT_SMD:SOT-223-3_TabPin2, symbol Regulator_Linear:NCP1117-3.3_SOT223
- added C35, C36, C37: 22u, Capacitor_SMD:C_0402_1005Metric, symbol Device:C
- added IC1: ISL91107IRTNZ-T, AAAAA:QFN50P300X400X80-21N, symbol AAAAAAA:ISL91107IRTNZ-T
- added L3: 1u, symbol Device:L
- D5: footprint (none) -> Diode_SMD:D_0402_1005Metric
- DS1: footprint (none) -> AAAAA:HIROSE_FH12S-40S-0.5SH_55_
Connections:
- net +3V3: now also C37.2, IC1.16 (FB), IC1.17 (VOUT_1), IC1.18 (VOUT_2), IC1.19 (VOUT_3), IC1.20 (VOUT_4)
- net GND: now also C35.1, C36.1, C37.1, IC1.15 (SGND), IC1.21 (EPAD), IC1.3 (PGND_1), IC1.4 (PGND_2)
- net Resistors should be close to microcontroller: now also J1.B5 (CC2), R6.1; no longer J1.A5 (CC1), R5.1
- net SW_C6: now also SW12.1, SW18.1, SW24.1, SW30.1, SW36.1, SW42.1, SW48.1, SW6.1
- net VSYS: now also C35.2, C36.2, IC1.10 (PVIN_4), IC1.12 (VIN), IC1.13 (EN), IC1.14 (MODE), IC1.7 (PVIN_1), IC1.8 (PVIN_2), IC1.9 (PVIN_3)
- new net: J1.A5 (CC1), R5.1
- new net: IC1.2 (LX2_2), L3.1
- new net: IC1.1 (LX2_1), L3.2
- no-connect marks 35 -> 37
Other:
- note added: "ISL91107IRTNZ buck/boost to 3.3V"
- note removed: "conversion to 3v3"
- moved on the sheet: J1, R5, R6

Commit message: screen, moving buttons
Connections:
- net GND: now also DS1.3 (IM0), DS1.34 (DOTCLK), DS1.35 (ENABLE), DS1.4 (IM1), DS1.5 (IM2), DS1.6 (IM3)
- net RDX: now reaches U5.28 (GPIO27)
- net RDX: now also DS1.13 (~{RDX})
- net WRX: now reaches U5.36 (GPIO28)
- net WRX: now also DS1.12 (~{WRX})
- net DCX: now reaches U5.37 (GPIO29)
- net DCX: now also DS1.11 (DCX)
- net CSX: now reaches U5.38 (GPIO30)
- net CSX: now also DS1.10 (~{CSX})
- net DISPLAY_RESET: now reaches U5.39 (GPIO31)
- net DISPLAY_RESET: now also DS1.38 (~{RESX})
- net DB0: now reaches U5.40 (GPIO32)
- net DB0: now also DS1.14 (DB0)
- net DB1: now reaches U5.42 (GPIO33)
- net DB1: now also DS1.15 (DB1)
- net DB2: now reaches U5.43 (GPIO34)
- net DB2: now also DS1.16 (DB2)
- net DB3: now reaches U5.44 (GPIO35)
- net DB3: now also DS1.17 (DB3)
- net DB4: now reaches U5.45 (GPIO36)
- net DB4: now also DS1.18 (DB4)
- net DB5: now reaches U5.46 (GPIO37)
- net DB5: now also DS1.19 (DB5)
- net DB6: now reaches U5.47 (GPIO38)
- net DB6: now also DS1.20 (DB6)
- net DB7: now reaches U5.48 (GPIO39)
- net DB7: now also DS1.21 (DB7)
- no-connect marks 37 -> 39
Other:
- note added: "80-8bit parallel I/F"
- note added: "active low"
- moved on the sheet: C1, C10, C11, C12, C13, C14, C15, C16, C17, C2, C28, C29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

Commit message: more moving things
Connections:
- net CSX: now also U5.1 (GPIO4); no longer U5.38 (GPIO30)
- net DB0: now also U5.6 (GPIO8); no longer U5.40 (GPIO32)
- net DB1: now also U5.7 (GPIO9); no longer U5.42 (GPIO33)
- net DB2: now also U5.8 (GPIO10); no longer U5.43 (GPIO34)
- net DB3: now also U5.9 (GPIO11); no longer U5.44 (GPIO35)
- net DB4: now also U5.11 (GPIO12); no longer U5.45 (GPIO36)
- net DB5: now also U5.12 (GPIO13); no longer U5.46 (GPIO37)
- net DB6: now also U5.13 (GPIO14); no longer U5.47 (GPIO38)
- net DB7: now also U5.14 (GPIO15); no longer U5.48 (GPIO39)
- net DCX: now also U5.2 (GPIO5); no longer U5.37 (GPIO29)
- net DISPLAY_RESET: now also U5.16 (GPIO16); no longer U5.39 (GPIO31)
- net RDX: now also U5.4 (GPIO7); no longer U5.28 (GPIO27)
- net SW_C1: now also U5.37 (GPIO29); no longer U5.7 (GPIO9)
- net SW_C2: now also U5.38 (GPIO30); no longer U5.8 (GPIO10)
- net SW_C3: now also U5.39 (GPIO31); no longer U5.9 (GPIO11)
- net SW_C4: now also U5.40 (GPIO32); no longer U5.11 (GPIO12)
- net SW_C5: now also U5.42 (GPIO33); no longer U5.12 (GPIO13)
- net SW_C6: now also U5.43 (GPIO34); no longer U5.13 (GPIO14)
- net SW_R1: now also U5.36 (GPIO28)
- net SW_R2: now also U5.28 (GPIO27)
- net SW_R3: now also U5.27 (GPIO26)
- net SW_R4: now also U5.21 (GPIO21); no longer U5.1 (GPIO4)
- net SW_R5: now also U5.22 (GPIO22); no longer U5.2 (GPIO5)
- net SW_R6: now also U5.23 (GPIO23); no longer U5.3 (GPIO6)
- net SW_R7: now also U5.25 (GPIO24); no longer U5.4 (GPIO7)
- net SW_R8: now also U5.26 (GPIO25); no longer U5.6 (GPIO8)
- net WRX: now also U5.3 (GPIO6); no longer U5.36 (GPIO28)
- no-connect marks 39 -> 29
Other:
- moved on the sheet: C1, C10, C11, C12, C13, C14, C15, C16, C17, C2, C3, C6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
