File: calc-v2.kicad_pcb (KiCad board)
At the start: 2 copper layers, 100 x 111.4 mm, 107 parts, among them IC1 ISL91107IRTNZ-T, J1 USB_C_Receptacle_USB2.0_16P, SW1 SW_Push_45deg, SW10 SW_Push_45deg, SW11 SW_Push_45deg, SW12 SW_Push_45deg, SW13 SW_Push_45deg, SW14 SW_Push_45deg, SW15 SW_Push_45deg, SW16 SW_Push_45deg, SW17 SW_Push_45deg, SW18 SW_Push_45deg, SW19 SW_Push_45deg, SW2 SW_Push_45deg, SW20 SW_Push_45deg, SW21 SW_Push_45deg, SW22 SW_Push_45deg, SW23 SW_Push_45deg, SW24 SW_Push_45deg, SW25 SW_Push_45deg, SW26 SW_Push_45deg, SW27 SW_Push_45deg, SW28 SW_Push_45deg, SW29 SW_Push_45deg, SW3 SW_Push_45deg, SW30 SW_Push_45deg, SW31 SW_Push_45deg, SW32 SW_Push_45deg, SW33 SW_Push_45deg, SW34 SW_Push_45deg, SW35 SW_Push_45deg, SW36 SW_Push_45deg, SW37 SW_Push_45deg, SW38 SW_Push_45deg, SW39 SW_Push_45deg, SW4 SW_Push_45deg, SW40 SW_Push_45deg, SW41 SW_Push_45deg, SW42 SW_Push_45deg, SW43 SW_Push_45deg, SW44 SW_Push_45deg, SW45 SW_Push_45deg, SW46 SW_Push_45deg, SW47 SW_Push_45deg, SW48 SW_Push_45deg, SW49 SW_Push_45deg, SW5 SW_Push_45deg, SW6 SW_Push_45deg, SW7 SW_Push_45deg, SW8 SW_Push_45deg, SW9 SW_Push_45deg, U1 W25Q128JVS, U2 TPS92200D2DDC, U3 BQ24074RGT, U5 RP2350B, U6 APS6404L-3SQRx-ZR, Y1 ABM8-272-T3

Commit message: afjlkasdfjkasd
Parts:
- removed C26, C27: 100n, Capacitor_SMD:C_0402_1005Metric
- removed C34: 1u, Capacitor_SMD:C_0402_1005Metric
- removed R10, R17: 10k, Resistor_SMD:R_0201_0603Metric
- removed R15: 1k, Resistor_SMD:R_0402_1005Metric
- removed U1: W25Q128JVS, Package_SO:SOIC-8_5.3x5.3mm_P1.27mm
- removed U6: APS6404L-3SQRx-ZR, Package_SON:Winbond_USON-8-1EP_3x2mm_P0.5mm_EP0.2x1.6mm
- added J2: Conn_01x02_MountingPin, Connector_JST:JST_PH_S2B-PH-SM4-TB_1x02-1MP_P2.00mm_Horizontal, B.Cu at (25.6, 125.7)
- J1: value USB_C_Receptacle_USB2.0_16P -> USB_C_Receptacle_USB2.0_14P; footprint Connector_USB:USB_C_Receptacle_Amphenol_124019772112A -> Connector_USB:USB_C_Receptacle_GCT_USB4105-xx-A_16P_TopMnt_Horizontal
- moved C35 83.7 mm to (39.4, 115.2), turned to 90 degrees
- moved C36 82.2 mm to (40.8, 115.2), turned to 90 degrees
- moved IC1 75.6 mm to (40.0, 111.0)
- moved L3 74.0 mm to (44.7, 110.0), turned to 90 degrees
- moved C37 71.9 mm to (36.5, 107.7), turned to 0 degrees
- moved SW49 57.7 mm to (16.1, 84.3)
- moved C24 57.5 mm to (20.4, 111.3), turned to 90 degrees
- moved C33 56.2 mm to (17.1, 115.9), turned to -90 degrees
- moved R8 51.7 mm to (14.4, 114.8), turned to 90 degrees
- moved C25 51.3 mm to (10.5, 110.9)
- moved R9 51.2 mm to (19.1, 112.7)
- moved R12 50.8 mm to (19.1, 109.0), turned to 0 degrees
- moved R13 50.1 mm to (19.0, 110.0)
- moved R11 49.1 mm to (15.5, 116.1), turned to 90 degrees
- moved U3 48.1 mm to (15.3, 111.5), turned to 0 degrees
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Connections:
- J1 pad A8: unconnected-(J1-SBU1-PadA8) -> (no net)
- J1 pad B8: unconnected-(J1-SBU1-PadA8) -> (no net)
- J1 pad SH: (no net) -> GND
- SW49 pad 1: Net-(R15-Pad2) -> GND
- SW49 pad 2: GND -> Net-(U5-~{QSPI_SS})
- U5 pad 19: unconnected-(U5-GPIO19-Pad19) -> PGOOD
- U5 pad 20: unconnected-(U5-GPIO20-Pad20) -> CHG
- U5 pad 21: SW_R4 -> unconnected-(U5-GPIO21-Pad21)
- U5 pad 22: SW_R5 -> unconnected-(U5-GPIO22-Pad22)
- U5 pad 23: SW_R6 -> unconnected-(U5-GPIO23-Pad23)
- U5 pad 44: unconnected-(U5-GPIO35-Pad44) -> SW_R4
- U5 pad 45: unconnected-(U5-GPIO36-Pad45) -> SW_R5
- U5 pad 46: unconnected-(U5-GPIO37-Pad46) -> SW_R6
- U5 pad 70: FLASH_IO3 -> unconnected-(U5-QSPI_SD3-Pad70)
- U5 pad 71: FLASH_SCLK -> unconnected-(U5-QSPI_SCLK-Pad71)
- U5 pad 72: FLASH_IO0 -> unconnected-(U5-QSPI_SD0-Pad72)
- U5 pad 73: FLASH_IO2 -> unconnected-(U5-QSPI_SD2-Pad73)
- U5 pad 74: FLASH_IO1 -> unconnected-(U5-QSPI_SD1-Pad74)
- U5 pad 75: FLASH_SS -> Net-(U5-~{QSPI_SS})
- U5 pad 77: PSRAM_SS -> unconnected-(U5-GPIO0-Pad77)
Routing:
- net GND: track 0.99 -> 184.4 mm, vias 0 -> 8
- net +3V3: track 5.27 -> 152.4 mm, vias 0 -> 7
- net VSYS: track 0.00 -> 53.1 mm, vias 0 -> 3
- net +1V1: track 0.00 -> 46.8 mm
- net DISPLAY_BCKLGHT: track 0.00 -> 31.2 mm
- net +BATT: track 0.00 -> 28.1 mm, vias 0 -> 1
- net XIN: track 0.00 -> 27.9 mm
- net CSX: track 0.00 -> 24.9 mm
- net SPI_RS: track 0.00 -> 24.5 mm, vias 0 -> 2
- net SPI_SCK: track 0.00 -> 23.4 mm
- net SW_C1: track 85.0 -> 65.3 mm
- net SW_C3: track 85.0 -> 102.6 mm
- net XOUT: track 0.00 -> 16.5 mm
- net USB_D-: track 0.00 -> 16.0 mm
- net USB_D+: track 0.00 -> 16.0 mm
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- added copper zone on B.Cu, net GND
